File: hardware/kicad/KEYPAD_4X4.kicad_sch (KiCad schematic)
At the start: 9 parts, among them J3 Conn_01x08_MountingPin

Commit message: fix: error fixing & connection config
Parts:
- renumbered R45 to R46, R44 to R47, R43 to R48, R42 to R49, R41 to R50, R40 to R51, R39 to R52, R38 to R53
Connections:
- no-connect marks 0 -> 1
Changed lines of the file:
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@@
 	(generator_version "9.0")
 	(paper "A4")
+	(no_connect
+		(at 179.07 73.66)
+	)
 	(wire
 		(pts
@@
 		(on_board yes)
 		(dnp no)
-		(property "Reference" "R38"
+		(property "Reference" "R53"
 			(at 170.688 72.39 0)
 			(effects
@@
 		(instances
 			(project ""
-				(path "/0357579f-0f06-4880-b651-8e2778a9baa9/89709966-3837-454c-8ae3-6689f2487bbb/cd523802-ff60-46d2-9bc3-ed925dd91a9c"
-					(reference "R38")
+				(path "/0357579f-0f06-4880-b651-8e2778a9baa9/89709966-3837-454c-8ae3-6689f2487bbb/1076efd2-bfaa-449f-bc2b-848a16dac785"
+					(reference "R53")
 					(unit 1)
 				)
@@
 		(on_board yes)
 		(dnp no)
-		(property "Reference" "R42"
+		(property "Reference" "R49"
 			(at 139.954 72.136 0)
 			(effects
@@
 		(instances
 			(project ""
-				(path "/0357579f-0f06-4880-b651-8e2778a9baa9/89709966-3837-454c-8ae3-6689f2487bbb/cd523802-ff60-46d2-9bc3-ed925dd91a9c"
-					(reference "R42")
+				(path "/0357579f-0f06-4880-b651-8e2778a9baa9/89709966-3837-454c-8ae3-6689f2487bbb/1076efd2-bfaa-449f-bc2b-848a16dac785"
+					(reference "R49")
 					(unit 1)
 				)
@@
 		(on_board yes)
 		(dnp no)
-		(property "Reference" "R40"
+		(property "Reference" "R51"
 			(at 155.448 72.39 0)
 			(effects
@@
 		(instances
 			(project ""
-				(path "/0357579f-0f06-4880-b651-8e2778a9baa9/89709966-3837-454c-8ae3-6689f2487bbb/cd523802-ff60-46d2-9bc3-ed925dd91a9c"
-					(reference "R40")
+				(path "/0357579f-0f06-4880-b651-8e2778a9baa9/89709966-3837-454c-8ae3-6689f2487bbb/1076efd2-bfaa-449f-bc2b-848a16dac785"
+					(reference "R51")
 					(unit 1)
 				)
@@
 		(on_board yes)
 		(dnp no)
-		(property "Reference" "R41"
+		(property "Reference" "R50"
 			(at 147.574 72.136 0)
 			(effects
@@
 		(instances
 			(project ""
-				(path "/0357579f-0f06-4880-b651-8e2778a9baa9/89709966-3837-454c-8ae3-6689f2487bbb/cd523802-ff60-46d2-9bc3-ed925dd91a9c"
-					(reference "R41")
+				(path "/0357579f-0f06-4880-b651-8e2778a9baa9/89709966-3837-454c-8ae3-6689f2487bbb/1076efd2-bfaa-449f-bc2b-848a16dac785"
+					(reference "R50")
 					(unit 1)
 				)
@@
 		(instances
 			(project ""
-				(path "/0357579f-0f06-4880-b651-8e2778a9baa9/89709966-3837-454c-8ae3-6689f2487bbb/cd523802-ff60-46d2-9bc3-ed925dd91a9c"
+				(path "/0357579f-0f06-4880-b651-8e2778a9baa9/89709966-3837-454c-8ae3-6689f2487bbb/1076efd2-bfaa-449f-bc2b-848a16dac785"
 					(reference "J3")
 					(unit 1)
@@
 		(on_board yes)
 		(dnp no)
-		(property "Reference" "R39"
+		(property "Reference" "R52"
 			(at 162.56 72.39 0)
 			(effects
@@
 		(instances
 			(project ""
-				(path "/0357579f-0f06-4880-b651-8e2778a9baa9/89709966-3837-454c-8ae3-6689f2487bbb/cd523802-ff60-46d2-9bc3-ed925dd91a9c"
-					(reference "R39")
+				(path "/0357579f-0f06-4880-b651-8e2778a9baa9/89709966-3837-454c-8ae3-6689f2487bbb/1076efd2-bfaa-449f-bc2b-848a16dac785"
+					(reference "R52")
 					(unit 1)
 				)
@@
 		(on_board yes)
 		(dnp no)
-		(property "Reference" "R44"
+		(property "Reference" "R47"
 			(at 124.714 72.39 0)
 			(effects
@@
 		(instances
 			(project ""
-				(path "/0357579f-0f06-4880-b651-8e2778a9baa9/89709966-3837-454c-8ae3-6689f2487bbb/cd523802-ff60-46d2-9bc3-ed925dd91a9c"
-					(reference "R44")
+				(path "/0357579f-0f06-4880-b651-8e2778a9baa9/89709966-3837-454c-8ae3-6689f2487bbb/1076efd2-bfaa-449f-bc2b-848a16dac785"
+					(reference "R47")
 					(unit 1)
 				)
@@
 		(on_board yes)
 		(dnp no)
-		(property "Reference" "R43"
+		(property "Reference" "R48"
 			(at 132.334 72.136 0)
 			(effects
@@
 		(instances
 			(project ""
-				(path "/0357579f-0f06-4880-b651-8e2778a9baa9/89709966-3837-454c-8ae3-6689f2487bbb/cd523802-ff60-46d2-9bc3-ed925dd91a9c"
-					(reference "R43")
+				(path "/0357579f-0f06-4880-b651-8e2778a9baa9/89709966-3837-454c-8ae3-6689f2487bbb/1076efd2-bfaa-449f-bc2b-848a16dac785"
+					(reference "R48")
 					(unit 1)
 				)
@@
 		(on_board yes)
 		(dnp no)
-		(property "Reference" "R45"
+		(property "Reference" "R46"
 			(at 116.84 72.39 0)
 			(effects
@@
 		(instances
 			(project ""
-				(path "/0357579f-0f06-4880-b651-8e2778a9baa9/89709966-3837-454c-8ae3-6689f2487bbb/cd523802-ff60-46d2-9bc3-ed925dd91a9c"
-					(reference "R45")
+				(path "/0357579f-0f06-4880-b651-8e2778a9baa9/89709966-3837-454c-8ae3-6689f2487bbb/1076efd2-bfaa-449f-bc2b-848a16dac785"
+					(reference "R46")
 					(unit 1)
 				)

Commit message: docs: added end semester report for project
Parts:
- J3: symbol Connector_Generic_MountingPin:Conn_01x08_MountingPin -> TPSM82903:Conn_01x08_MountingPin
- R46, R47, R48, R49, R50, R51, R52, R53: symbol Device:R -> TPSM82903:R
Changed lines of the file:
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@@
 	)
 	(symbol
-		(lib_id "Device:R")
+		(lib_id "TPSM82903:R")
 		(at 168.91 73.66 0)
 		(unit 1)
@@
 	)
 	(symbol
-		(lib_id "Device:R")
+		(lib_id "TPSM82903:R")
 		(at 138.43 73.66 0)
 		(unit 1)
@@
 	)
 	(symbol
-		(lib_id "Device:R")
+		(lib_id "TPSM82903:R")
 		(at 153.67 73.66 0)
 		(unit 1)
@@
 	)
 	(symbol
-		(lib_id "Device:R")
+		(lib_id "TPSM82903:R")
 		(at 146.05 73.66 0)
 		(unit 1)
@@
 	)
 	(symbol
-		(lib_id "Connector_Generic_MountingPin:Conn_01x08_MountingPin")
+		(lib_id "TPSM82903:Conn_01x08_MountingPin")
 		(at 179.07 58.42 0)
 		(unit 1)
@@
 	)
 	(symbol
-		(lib_id "Device:R")
+		(lib_id "TPSM82903:R")
 		(at 161.29 73.66 0)
 		(unit 1)
@@
 	)
 	(symbol
-		(lib_id "Device:R")
+		(lib_id "TPSM82903:R")
 		(at 123.19 73.66 0)
 		(unit 1)
@@
 	)
 	(symbol
-		(lib_id "Device:R")
+		(lib_id "TPSM82903:R")
 		(at 130.81 73.66 0)
 		(unit 1)
@@
 	)
 	(symbol
-		(lib_id "Device:R")
+		(lib_id "TPSM82903:R")
 		(at 115.57 73.66 0)
 		(unit 1)
