File: hardware/kicad/card_issuance_power.kicad_sch (KiCad schematic)
At the start: 17 parts, among them J2 Conn_01x02_Pin, Q1 IRF4905

Commit message: feat: separated modules but added power module
Parts:
- added J2, J3, J4: Conn_01x02_Pin, Terminal Blocks:CONN_PM 5.08&slash_02&slash_90 3.5SN BK BX_WED, symbol Connector:Conn_01x02_Pin
- R1, R2, R3, R4, R5: footprint (none) -> Resistor_THT:R_Axial_DIN0207_L6.3mm_D2.5mm_P2.54mm_Vertical
- renumbered J2 to J1
Connections:
- net GND_LOGIC: now also R2.2, J3.2 (Pin_2), J4.2 (Pin_2); no longer R3.2
- net GND_MOTOR: now also R3.2, J2.2 (Pin_2); no longer R2.2
- net V12_MOTOR: no longer names the net of C3.1, F2.2
- net V12_MOTOR: now also J2.1 (Pin_1)
- new net BUCK_3V3/VOUT: J3.1 (Pin_1)
- new net BUCK_5.1/VOUT: J4.1 (Pin_1)
Other:
- sheet BUCK_3V3 ports: added GND; removed none
- sheet BUCK_5.1 ports: added GND; removed none
- moved on the sheet: C1, C2, C3, C4, D1, F1, F2, F3, J1, Q1, R1, R2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

Commit message: fix: buck connections
Parts:
- D1: footprint (none) -> Diode_THT:D_DO-41_SOD81_P10.16mm_Horizontal
- F1, F2, F3: footprint (none) -> Fuse:Fuse_Blade_Mini_directSolder
- J1: value Conn_01x02_Pin -> V12_IN; footprint Terminal Blocks:CONN_PM 5.08&slash_02&slash_90 3.5SN BK BX_WED -> Terminals:CONN_PM 5.08&slash_02&slash_90 3.5SN BK BX_WED
- J2: value Conn_01x02_Pin -> V12_OUT; footprint Terminal Blocks:CONN_PM 5.08&slash_02&slash_90 3.5SN BK BX_WED -> Terminals:CONN_PM 5.08&slash_02&slash_90 3.5SN BK BX_WED
- J3: value Conn_01x02_Pin -> V3V3_OUT; footprint Terminal Blocks:CONN_PM 5.08&slash_02&slash_90 3.5SN BK BX_WED -> Terminals:CONN_PM 5.08&slash_02&slash_90 3.5SN BK BX_WED
- J4: value Conn_01x02_Pin -> V5.1_OUT; footprint Terminal Blocks:CONN_PM 5.08&slash_02&slash_90 3.5SN BK BX_WED -> Terminals:CONN_PM 5.08&slash_02&slash_90 3.5SN BK BX_WED
Changed lines of the file:
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@@
 			)
 		)
-		(property "Value" "Conn_01x02_Pin"
+		(property "Value" "V12_IN"
 			(at 42.545 59.69 0)
 			(effects
@@
 			)
 		)
-		(property "Footprint" "Terminal Blocks:CONN_PM 5.08&slash_02&slash_90 3.5SN BK BX_WED"
+		(property "Footprint" "Terminals:CONN_PM 5.08&slash_02&slash_90 3.5SN BK BX_WED"
 			(at 41.91 62.23 0)
 			(effects
@@
 			)
 		)
-		(property "Value" "Conn_01x02_Pin"
+		(property "Value" "V5.1_OUT"
 			(at 260.35 69.8499 0)
 			(effects
@@
 			)
 		)
-		(property "Footprint" "Terminal Blocks:CONN_PM 5.08&slash_02&slash_90 3.5SN BK BX_WED"
+		(property "Footprint" "Terminals:CONN_PM 5.08&slash_02&slash_90 3.5SN BK BX_WED"
 			(at 259.08 67.31 0)
 			(effects
@@
 			)
 		)
-		(property "Value" "Conn_01x02_Pin"
+		(property "Value" "V3V3_OUT"
 			(at 260.35 55.8799 0)
 			(effects
@@
 			)
 		)
-		(property "Footprint" "Terminal Blocks:CONN_PM 5.08&slash_02&slash_90 3.5SN BK BX_WED"
+		(property "Footprint" "Terminals:CONN_PM 5.08&slash_02&slash_90 3.5SN BK BX_WED"
 			(at 259.08 53.34 0)
 			(effects
@@
 			)
 		)
-		(property "Value" "Conn_01x02_Pin"
+		(property "Value" "V12_OUT"
 			(at 191.77 49.5299 0)
 			(effects
@@
 			)
 		)
-		(property "Footprint" "Terminal Blocks:CONN_PM 5.08&slash_02&slash_90 3.5SN BK BX_WED"
+		(property "Footprint" "Terminals:CONN_PM 5.08&slash_02&slash_90 3.5SN BK BX_WED"
 			(at 190.5 46.99 0)
 			(effects
@@
 			)
 		)
-		(property "Footprint" ""
+		(property "Footprint" "Fuse:Fuse_Blade_Mini_directSolder"
 			(at 55.88 56.388 90)
 			(effects
@@
 			)
 		)
-		(property "Footprint" ""
+		(property "Footprint" "Diode_THT:D_DO-41_SOD81_P10.16mm_Horizontal"
 			(at 66.04 60.96 0)
 			(effects
@@
 			)
 		)
-		(property "Footprint" ""
+		(property "Footprint" "Fuse:Fuse_Blade_Mini_directSolder"
 			(at 161.29 71.628 90)
 			(effects
@@
 			)
 		)
-		(property "Footprint" ""
+		(property "Footprint" "Fuse:Fuse_Blade_Mini_directSolder"
 			(at 161.29 48.768 90)
 			(effects

Commit message: feat: added settings - pcb design
Connections:
- net V12_PROT: now reaches C1.1, C2.1, F2.1, F3.1, Q1.2 (D)
- net GND_STAR: now reaches C1.2, C2.2, J1.2 (Pin_2), R1.2, R2.1, R3.1, TP2.1
- net V12_PROT_12V: now reaches C3.1, F2.2, J2.1 (Pin_1)
- net V12_IN: now reaches F1.1, J1.1 (Pin_1), TP1.1
- net V12_FUSED: now reaches D1.2 (A), F1.2, Q1.3 (S), R4.1
- net BUCK_3V3/VIN renamed V12_PROT_5V
- net BUCK_3V3/VOUT renamed V3V3_OUT
- net BUCK_5.1/VOUT renamed V5.1_OUT
Other:
- moved on the sheet: J3, J4
Changed lines of the file:
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@@
 	)
 	(junction
-		(at 251.46 62.23)
+		(at 250.19 62.23)
 		(diameter 0)
 		(color 0 0 0 0)
@@
 	(wire
 		(pts
-			(xy 251.46 62.23) (xy 251.46 69.85)
+			(xy 250.19 62.23) (xy 250.19 69.85)
 		)
 		(stroke
@@
 	(wire
 		(pts
-			(xy 251.46 55.88) (xy 254 55.88)
+			(xy 250.19 55.88) (xy 260.35 55.88)
 		)
 		(stroke
@@
 	(wire
 		(pts
-			(xy 251.46 69.85) (xy 254 69.85)
-		)
-		(stroke
-			(width 0)
-			(type default)
-		)
-	)
-	(wire
-		(pts
-			(xy 247.65 67.31) (xy 254 67.31)
+			(xy 250.19 69.85) (xy 260.35 69.85)
 		)
 		(stroke
@@
 	(wire
 		(pts
-			(xy 251.46 62.23) (xy 251.46 55.88)
+			(xy 250.19 62.23) (xy 250.19 55.88)
 		)
 		(stroke
@@
 	(wire
 		(pts
-			(xy 224.79 62.23) (xy 251.46 62.23)
+			(xy 224.79 62.23) (xy 250.19 62.23)
 		)
 		(stroke
@@
 	(wire
 		(pts
-			(xy 247.65 53.34) (xy 254 53.34)
+			(xy 247.65 53.34) (xy 260.35 53.34)
+		)
+		(stroke
+			(width 0)
+			(type default)
+		)
+	)
+	(wire
+		(pts
+			(xy 247.65 67.31) (xy 260.35 67.31)
 		)
 		(stroke
@@
 			(width 0)
 			(type default)
+		)
+	)
+	(label "V12_IN"
+		(at 46.99 62.23 0)
+		(effects
+			(font
+				(size 1.27 1.27)
+			)
+			(justify left bottom)
+		)
+	)
+	(label "V12_PROT_5V"
+		(at 181.61 62.23 0)
+		(effects
+			(font
+				(size 1.27 1.27)
+			)
+			(justify left bottom)
+		)
+	)
+	(label "V12_FUSED"
+		(at 76.2 54.61 0)
+		(effects
+			(font
+				(size 1.27 1.27)
+			)
+			(justify left bottom)
+		)
+	)
+	(label "V12_PROT"
+		(at 93.98 76.2 0)
+		(effects
+			(font
+				(size 1.27 1.27)
+			)
+			(justify left bottom)
+		)
+	)
+	(label "V3V3_OUT"
+		(at 251.46 53.34 0)
+		(effects
+			(font
+				(size 1.27 1.27)
+			)
+			(justify left bottom)
+		)
+	)
+	(label "V5.1_OUT"
+		(at 251.46 67.31 0)
+		(effects
+			(font
+				(size 1.27 1.27)
+			)
+			(justify left bottom)
 		)
 	)
@@
 	(label "GND_LOGIC"
 		(at 63.5 72.39 0)
+		(effects
+			(font
+				(size 1.27 1.27)
+			)
+			(justify left bottom)
+		)
+	)
+	(label "GND_STAR"
+		(at 46.99 64.77 0)
+		(effects
+			(font
+				(size 1.27 1.27)
+			)
+			(justify left bottom)
+		)
+	)
+	(label "V12_PROT_12V"
+		(at 170.18 46.99 0)
 		(effects
 			(font
@@
 	(symbol
 		(lib_id "Connector:Conn_01x02_Pin")
-		(at 259.08 67.31 0)
+		(at 265.43 67.31 0)
 		(mirror y)
 		(unit 1)
@@
 		(fields_autoplaced yes)
 		(property "Reference" "J4"
-			(at 260.35 67.3099 0)
+			(at 266.7 67.3099 0)
 			(effects
 				(font
@@
 		)
 		(property "Value" "V5.1_OUT"
-			(at 260.35 69.8499 0)
+			(at 266.7 69.8499 0)
 			(effects
 				(font
@@
 		)
 		(property "Footprint" "Terminals:CONN_PM 5.08&slash_02&slash_90 3.5SN BK BX_WED"
-			(at 259.08 67.31 0)
+			(at 265.43 67.31 0)
 			(effects
 				(font
@@
 		)
 		(property "Datasheet" "~"
-			(at 259.08 67.31 0)
+			(at 265.43 67.31 0)
 			(effects
 				(font
@@
 		)
 		(property "Description" "Generic connector, single row, 01x02, script generated"
-			(at 259.08 67.31 0)
+			(at 265.43 67.31 0)
 			(effects
 				(font
@@
 	(symbol
 		(lib_id "Connector:Conn_01x02_Pin")
-		(at 259.08 53.34 0)
+		(at 265.43 53.34 0)
 		(mirror y)
 		(unit 1)
@@
 		(fields_autoplaced yes)
 		(property "Reference" "J3"
-			(at 260.35 53.3399 0)
+			(at 266.7 53.3399 0)
 			(effects
 				(font
@@
 		)
 		(property "Value" "V3V3_OUT"
-			(at 260.35 55.8799 0)
+			(at 266.7 55.8799 0)
 			(effects
 				(font
@@
 		)
 		(property "Footprint" "Terminals:CONN_PM 5.08&slash_02&slash_90 3.5SN BK BX_WED"
-			(at 259.08 53.34 0)
+			(at 265.43 53.34 0)
 			(effects
 				(font
@@
 		)
 		(property "Datasheet" "~"
-			(at 259.08 53.34 0)
+			(at 265.43 53.34 0)
 			(effects
 				(font
@@
 		)
 		(property "Description" "Generic connector, single row, 01x02, script generated"
-			(at 259.08 53.34 0)
-			(effects
-				(font
+			(at 265.43 53.34 0)
+			(effects
+				(font

Commit message: chore: pcb planes filling & vias
Connections:
- net GND_LOGIC: no longer F3.2
- net V12_FUSED: now also TP1.1
- net V12_IN: no longer TP1.1
- net V12_PROT_5V: now also F3.2
Other:
- moved on the sheet: TP1
Changed lines of the file:
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@@
-	)
-	(junction
-		(at 170.18 69.85)
-		(diameter 0)
-		(color 0 0 0 0)
 	)
 	(junction
@@
 	)
 	(junction
+		(at 170.18 59.69)
+		(diameter 0)
+		(color 0 0 0 0)
+	)
+	(junction
 		(at 153.67 58.42)
 		(diameter 0)
@@
 		(color 0 0 0 0)
 	)
-	(junction
-		(at 50.8 54.61)
-		(diameter 0)
-		(color 0 0 0 0)
-	)
 	(wire
 		(pts
@@
 	(wire
 		(pts
-			(xy 45.72 54.61) (xy 50.8 54.61)
-		)
-		(stroke
-			(width 0)
-			(type default)
-		)
-	)
-	(wire
-		(pts
 			(xy 66.04 54.61) (xy 76.2 54.61)
 		)
@@
 	(wire
 		(pts
+			(xy 66.04 52.07) (xy 66.04 54.61)
+		)
+		(stroke
+			(width 0)
+			(type default)
+		)
+	)
+	(wire
+		(pts
 			(xy 93.98 76.2) (xy 93.98 69.85)
 		)
@@
 	(wire
 		(pts
-			(xy 165.1 69.85) (xy 170.18 69.85)
-		)
-		(stroke
-			(width 0)
-			(type default)
-		)
-	)
-	(wire
-		(pts
 			(xy 223.52 52.07) (xy 223.52 62.23)
 		)
@@
 	(wire
 		(pts
+			(xy 166.37 59.69) (xy 170.18 59.69)
+		)
+		(stroke
+			(width 0)
+			(type default)
+		)
+	)
+	(wire
+		(pts
 			(xy 76.2 64.77) (xy 77.47 64.77)
 		)
@@
 		(pts
 			(xy 50.8 54.61) (xy 52.07 54.61)
+		)
+		(stroke
+			(width 0)
+			(type default)
+		)
+	)
+	(wire
+		(pts
+			(xy 165.1 69.85) (xy 166.37 69.85)
+		)
+		(stroke
+			(width 0)
+			(type default)
+		)
+	)
+	(wire
+		(pts
+			(xy 166.37 69.85) (xy 166.37 59.69)
 		)
 		(stroke
@@
 	(symbol
 		(lib_id "Connector:TestPoint")
-		(at 45.72 54.61 90)
+		(at 66.04 52.07 0)
 		(unit 1)
 		(exclude_from_sim no)
@@
 		(dnp no)
 		(property "Reference" "TP1"
-			(at 42.164 50.038 90)
+			(at 62.992 48.768 0)
 			(effects
 				(font
@@
 		)
 		(property "Value" "V12_IN"
-			(at 42.164 52.578 90)
+			(at 61.722 50.546 0)
 			(effects
 				(font
@@
 		)
 		(property "Footprint" "TestPoint:TestPoint_THTPad_2.0x2.0mm_Drill1.0mm"
-			(at 45.72 49.53 0)
+			(at 71.12 52.07 0)
 			(effects
 				(font
@@
 		)
 		(property "Datasheet" "~"
-			(at 45.72 49.53 0)
+			(at 71.12 52.07 0)
 			(effects
 				(font
@@
 		)
 		(property "Description" "test point"
-			(at 45.72 54.61 0)
-			(effects
-				(font
+			(at 66.04 52.07 0)
+			(effects
+				(font
